Commit message: updated obj files

File: Z1Env/robots/z1.urdf (robot description, URDF)
Before this commit: robot z1, 9 links, 8 joints
Links:
- link gripperMover: geometry collision mesh filename=package://robots/meshes/collision/z1_GripperMover.STL scale=1 1 1; visual mesh filename=package://robots/meshes/visual/z1_gripper_mover.obj scale=1 1 1
- link gripperStator: geometry collision mesh filename=package://robots/meshes/collision/z1_GripperStator.STL scale=1 1 1; visual mesh filename=package://robots/meshes/visual/z1_gripper_stator.obj scale=1 1 1
- link link0: geometry collision cylinder length=0.051 radius=0.0325; visual mesh filename=package://robots/meshes/visual/z1_link0.obj scale=1 1 1
- link link1: geometry visual mesh filename=package://robots/meshes/visual/z1_link1.obj scale=1 1 1
- link link2: geometry collision cylinder length=0.051 radius=0.0325; collision cylinder length=0.102 radius=0.0325
- link link3: geometry collision cylinder length=0.059 radius=0.0325; collision cylinder length=0.116 radius=0.02
- link link4: geometry collision cylinder length=0.067 radius=0.0325; visual mesh filename=package://robots/meshes/visual/z1_link4.obj scale=1 1 1
- link link5: geometry visual mesh filename=package://robots/meshes/visual/z1_link5.obj scale=1 1 1
- link link6: geometry collision cylinder length=0.051 radius=0.0325; visual mesh filename=package://robots/meshes/visual/z1_link6.obj scale=1 1 1

Commit message: added z1 env

File: Z1Env/robots/z1.urdf (robot description, URDF)
Before this commit: robot z1, 9 links, 8 joints
Joints:
- joint gripperStator: parent link06 -> link6
- joint joint1: child link01 -> link1; parent link00 -> link0
- joint joint2: child link02 -> link2; parent link01 -> link1
- joint joint3: child link03 -> link3; parent link02 -> link2
- joint joint4: child link04 -> link4; parent link03 -> link3
- joint joint5: child link05 -> link5; parent link04 -> link4
- joint joint6: child link06 -> link6; parent link05 -> link5

Commit message: updated urdf

File: Z1Env/robots/z1.urdf (robot description, URDF)
Before this commit: robot z1, 9 links, 8 joints
Joints:
- joint gripperStator: origin xyz=0.051 0.0 0.0 rpy=0 0 0 -> xyz=0.051 0.0 0.0 rpy=1.5708 0 0
- joint jointGripper: axis 0 1 0 -> 0 0 -1

Commit message: updated URDF

File: Z1Env/robots/z1.urdf (robot description, URDF)
Before this commit: robot z1, 9 links, 8 joints
Joints:
- joint gripperStator: origin xyz=0.051 0.0 0.0 rpy=1.5708 0 0 -> xyz=0.051 0.0 0.0 rpy=0 0 0
- joint jointGripper: axis 0 0 -1 -> 0 1 0

Commit message: added tcp link

File: Z1Env/robots/z1.urdf (robot description, URDF)
Before this commit: robot z1, 9 links, 8 joints
Links:
- added link tcp_link, mass 1e-5
Joints:
- added joint tcp_joint: type fixed, parent link6, child tcp_link, origin xyz=0.19 0.0 -0.01 rpy=0 0 0

Commit message: updated stl files

File: Z1Env/robots/z1.urdf (robot description, URDF)
Before this commit: robot z1, 10 links, 9 joints
Links:
- link link0: geometry collision mesh filename=package://robots/meshes/collision/z1_link0.STL scale=1 1 1; visual mesh filename=package://robots/meshes/visual/z1_link0.obj scale=1 1 1
- link link1: geometry collision mesh filename=package://robots/meshes/collision/z1_link1.STL scale=1 1 1; visual mesh filename=package://robots/meshes/visual/z1_link1.obj scale=1 1 1
- link link2: geometry collision mesh filename=package://robots/meshes/collision/z1_link2.STL scale=1 1 1; visual mesh filename=package://robots/meshes/visual/z1_link2.obj scale=1 1 1
- link link5: geometry collision mesh filename=package://robots/meshes/collision/z1_link5.STL scale=1 1 1; visual mesh filename=package://robots/meshes/visual/z1_link5.obj scale=1 1 1

Commit message: fixed shaking problem

File: Z1Env/robots/z1.urdf (robot description, URDF)
Before this commit: robot z1, 10 links, 9 joints
Links:
- link tcp_link: mass 1e-5 -> 1e-10

Commit message: updated collisions with stl files

File: Z1Env/robots/z1.urdf (robot description, URDF)
Before this commit: robot z1, 10 links, 9 joints
Links:
- link gripperMover: geometry collision mesh filename=package://robots/meshes/collision/z1_gripper_mover.STL scale=1 1 1; visual mesh filename=package://robots/meshes/visual/z1_gripper_mover.obj scale=1 1 1
- link gripperStator: geometry collision mesh filename=package://robots/meshes/collision/z1_gripper_stator.STL scale=1 1 1; visual mesh filename=package://robots/meshes/visual/z1_gripper_stator.obj scale=1 1 1
- link link3: geometry collision mesh filename=package://robots/meshes/collision/z1_link3.STL scale=1 1 1; visual mesh filename=package://robots/meshes/visual/z1_link3.obj scale=1 1 1
- link link4: geometry collision mesh filename=package://robots/meshes/collision/z1_link4.STL scale=1 1 1; visual mesh filename=package://robots/meshes/visual/z1_link4.obj scale=1 1 1
- link link6: geometry collision mesh filename=package://robots/meshes/collision/z1_link6.STL scale=1 1 1; visual mesh filename=package://robots/meshes/visual/z1_link6.obj scale=1 1 1
