Commit message: added gripper env

File: Z1Env/robots/gripper.urdf (robot description, URDF)
Before this commit: robot z1_gripper, 3 links, 2 joints
Links:
- added link link6, mass 0.28875807; collision mesh filename=package://robots/meshes/collision/z1_link6.STL scale=1 1 1; visual mesh filename=package://robots/meshes/visual/z1_link6.obj scale=1 1 1
Joints:
- added joint gripperStator: type fixed, parent link6, child gripperStator, origin xyz=0.051 0.0 0.0 rpy=0 0 0
